File: Version 1/D52M Feather Wing.kicad_pcb (KiCad board)
At the start: 2 copper layers, 22.9 x 50.8 mm, 2 parts, among them U1 ESP32FEATHER, U2 D52MxxM8

Commit message: Added version number to board and Kicad screenshot
Other:
- board text added: "Version 1"
Changed lines of the file:
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@@
   (general
     (thickness 1.6)
-    (drawings 13)
+    (drawings 14)
     (tracks 82)
     (zones 0)
@@
       (net 44 /BR2))
   )
+  (gr_text "Version 1" (at 0.635 -2.2225) (layer B.SilkS)
+    (effects (font (size 1.5 1.5) (thickness 0.3)) (justify mirror))
+  )
   (gr_text "Reegan McAllister\nCurtis Malainey" (at 0 1.27) (layer B.SilkS)
